File: Kiacd/MZ-2000_SD+NRF.kicad_pcb (KiCad board)
At the start: 2 copper layers, 115.8 x 142.7 mm, 21 parts, among them J1 Conn_02x22_Row_Letter_First, J2 RP2350B Left, J3 RP2350B Right, J4 VGA, J5 Micro_SD_Card_Kit, J6 MicroSD Card Adapter, U1 74LS04, U2 74LS30, U3 8255, U4 Arduino_Pro_Mini_5V

Commit message: Add files via upload
Parts:
- added D1: BAT54, Diode_THT:D_DO-41_SOD81_P10.16mm_Horizontal, F.Cu at (143.7, 150.4)
Connections:
- J2 pad 1: +5V -> (no net)
- J2 pad 16: (no net) -> Net-(D1-Pad1)
Routing:
- net Net-(D1-Pad1): track 0.00 -> 8.12 mm
- net +5V: track 295.3 -> 295.1 mm, vias 0 -> 1
Other:
- board text added: "1N5819"
- board text added: "MZ-2000_SD+NiseRamFile Rev1.1"
- board text removed: "MZ-2000_SD+NiseRamFile Rev1.0"
