File: Kiacd/MZ-2000_SD+NRF.sch (KiCad schematic (older format))
At the start: 17 parts, among them J1 Conn_02x22_Row_Letter_First, J2 RP2350B Left, J3 RP2350B Right, J4 VGA, J5 Micro_SD_Card_Kit, J6 MicroSD Card Adapter, U1 74LS04, U2 74LS30, U3 8255, U4 Arduino_Pro_Mini_5V

Commit message: Add files via upload
Parts:
- added D1: 1N5819, Diode_THT:D_DO-41_SOD81_P10.16mm_Horizontal, symbol Device:D
Changed lines of the file:
@@
 Title "MZ-2000_SD+NRF"
 Date ""
-Rev "Rev1.0"
+Rev "Rev1.1"
 Comp ""
 Comment1 ""
@@
 $EndComp
 Wire Wire Line
-	2500 5500 2100 5500
-Text Label 2100 5500 0    50   ~ 0
+	3500 5500 3300 5500
+Text Label 3350 5500 0    50   ~ 0
 +5V
 Text Label 2100 5900 0    50   ~ 0
@@
 NoConn ~ 2500 5600
 NoConn ~ 2500 5700
-NoConn ~ 3000 5500
 NoConn ~ 3000 5600
 NoConn ~ 5400 5550
@@
 Connection ~ 3950 8800
 Connection ~ 3950 10000
+NoConn ~ 2500 5500
+$Comp
+L Device:D D1
+U 1 1 6A1ABE9C
+P 3150 5500
+F 0 "D1" H 3150 5717 50  0000 C CNN
+F 1 "1N5819" H 3150 5626 50  0000 C CNN
+F 2 "Diode_THT:D_DO-41_SOD81_P10.16mm_Horizontal" H 3150 5500 50  0001 C CNN
+F 3 "~" H 3150 5500 50  0001 C CNN
+	1    3150 5500
+	1    0    0    -1
+$EndComp
 $EndSCHEMATC
